Commit message: first change

File: src/gazebo_test/model/robot.xacro (robot description, xacro)
@@ -20,5 +20,5 @@
 					<mesh filename="file://$(find gazebo_test)/model/aruco_work.dae"/>
 				</geometry>
-				<origin rpy="0 0 0" xyz="0 0 1"/> <!--Chaning xyz makes the move to exact position, defies gravity -->
+				<origin rpy="0 0 0" xyz="0 0 0"/> <!--Chaning xyz makes the move to exact position, defies gravity -->
 			</visual>
 			<collision>
